File: Hardware/KiCad/UV-Controller/UV-Controller.kicad_pcb (KiCad board)
At the start: 2 copper layers, 61 x 60 mm, 42 parts, among them IC1 W25Q16JVUXIQ_TR, J1 Conn_01x03_Socket, J2 Power Conn, J3 PWM Conn, J4 Conn, J5 Conn, SW1 SW_Push, SW2 SW_Push, U1 RP2040, U2 PEC16-4220F-S0024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

Commit message: Prepared gerbers for prod
Parts:
- added kibuzzard-67EEDD31: G***, kibuzzard-67EEDD31, F.Cu at (150.5, 106.7)
- added kibuzzard-67EEDD44: G***, kibuzzard-67EEDD44, F.Cu at (160.9, 106.7)
- added kibuzzard-67EEDF74: G***, kibuzzard-67EEDF74, B.Cu at (170.9, 86.0)
- added kibuzzard-67EEDFA4: G***, kibuzzard-67EEDFA4, B.Cu at (175.0, 86.0)
- added kibuzzard-67EEDFD5: G***, kibuzzard-67EEDFD5, B.Cu at (175.1, 99.8)
- added kibuzzard-67EEDFDD: G***, kibuzzard-67EEDFDD, B.Cu at (170.6, 99.8)
- added kibuzzard-67EEDFDD: G***, kibuzzard-67EEDFDD, B.Cu at (169.4, 78.0)
- added kibuzzard-67EEDFE5: G***, kibuzzard-67EEDFE5, B.Cu at (170.9, 95.2)
- added kibuzzard-67EEDFEA: G***, kibuzzard-67EEDFEA, B.Cu at (175.0, 95.2)
- added kibuzzard-67EEE001: G***, kibuzzard-67EEE001, B.Cu at (174.8, 90.5)
- added kibuzzard-67EEE00C: G***, kibuzzard-67EEE00C, B.Cu at (170.9, 90.5)
- added kibuzzard-67EEE0EE: G***, kibuzzard-67EEE0EE, B.Cu at (174.2, 78.0)
- added kibuzzard-67EEE147: G***, kibuzzard-67EEE147, B.Cu at (175.1, 105.8)
- added kibuzzard-67EEE14D: G***, kibuzzard-67EEE14D, B.Cu at (175.1, 110.6)
- added kibuzzard-67EEE153: G***, kibuzzard-67EEE153, B.Cu at (175.1, 115.1)
- moved R7 0.23 mm to (145.7, 88.2)
Routing:
- net GND: track 8.67 -> 9.95 mm, vias 65 -> 67
- net /CS: track 44.9 -> 44.1 mm
Other:
- board text added: "UV Lamp Controller By Szymon Wąchała For Nati <3 February 2025 v2.0"
