File: Hardware/KiCad/UV-Lamp/UV-Lamp.kicad_pcb (KiCad board)
At the start: 2 copper layers, 64 x 97 mm, 53 parts, among them IC1 LM3409HVMY, IC2 LM3409HVMY, J1 Conn, J2 Conn, J3 Connector, J4 Connector, J5 Conn, Q1 DMP10H400SK3-13, Q2 DMP10H400SK3-13, U1 TPS54560BDDA

Commit message: Prepared gerbers for prod
Routing:
- net GND: track 0.00 -> 2.61 mm
- net +48V: track 82.6 -> 81.9 mm
Other:
- board text added: "UV Lamp Power Board By Szymon Wąchała For Nati <3 March 2025 v2.0"
