File: Hardware/KiCad/UV-Lamp/UV-Lamp.kicad_sch (KiCad schematic)
At the start: 3 parts

Commit message: Prepared gerbers for prod
Changed lines of the file:
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@@
 	)
 	(sheet
-		(at 106.68 76.2)
+		(at 107.95 76.2)
 		(size 31.75 31.75)
 		(fields_autoplaced yes)
@@
 		)
 		(property "Sheetname" "Power Section"
-			(at 106.68 75.4884 0)
+			(at 107.95 75.4884 0)
 			(effects
 				(font
@@
 		)
 		(property "Sheetfile" "power-section.kicad_sch"
-			(at 106.68 108.5346 0)
+			(at 107.95 108.5346 0)
 			(effects
 				(font
@@
 	)
 	(sheet
-		(at 151.13 74.93)
-		(size 32.385 31.75)
+		(at 152.4 76.2)
+		(size 31.75 31.75)
 		(fields_autoplaced yes)
 		(stroke
@@
 		)
 		(property "Sheetname" "LED Driver"
-			(at 151.13 74.2184 0)
+			(at 152.4 75.4884 0)
 			(effects
 				(font
@@
 		)
 		(property "Sheetfile" "led-driver.kicad_sch"
-			(at 151.13 107.2646 0)
+			(at 152.4 108.5346 0)
 			(effects
 				(font
